File: git_testing.sch (KiCad schematic (older format))
At the start: 2 parts

Commit message: Update git_testing.sch
Parts:
- added MES?: Amperemeter_AC, symbol Device:Amperemeter_AC
- added R?: R, symbol Device:R
Changed lines of the file:
@@
+	1    0    0    -1
+$EndComp
+$Comp
+L Device:Amperemeter_AC MES?
+U 1 1 61166E32
+P 2700 2150
+F 0 "MES?" H 2853 2196 50  0000 L CNN
+F 1 "Amperemeter_AC" H 2853 2105 50  0000 L CNN
+F 2 "" V 2700 2250 50  0001 C CNN
+F 3 "~" V 2700 2250 50  0001 C CNN
+	1    2700 2150
+	1    0    0    -1
+$EndComp
+$Comp
+L Device:R R?
+U 1 1 6116760E
+P 6700 2250
+F 0 "R?" H 6770 2296 50  0000 L CNN
+F 1 "R" H 6770 2205 50  0000 L CNN
+F 2 "" V 6630 2250 50  0001 C CNN
+F 3 "~" H 6700 2250 50  0001 C CNN
+	1    6700 2250
 	1    0    0    -1
 $EndComp
